File: EAGLE/LoRa_Dev_revA.1/LoRa_Dev_A.1.sch (EAGLE design)
At the start: 28 parts, among them IC1 HMC8038LP4CETR, IC2 SX1262IMLTRT, J1 U.FL-R-SMT-1_80_, J2 HEADER_12PIN

Commit message: LoRa Silkscreen
Silkscreen and gerber files added
Parts:
- L1: value (none) -> 47nH
- Y1: value (none) -> 32MHz
Changed lines of the file:
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@@
 <part name="C5" library="NSE LABS" deviceset="C_0402" device="" value="5.6pF"/>
 <part name="SUPPLY10" library="supply2" library_urn="urn:adsk.eagle:library:372" deviceset="GND" device=""/>
-<part name="L1" library="NSE LABS" deviceset="L_0603" device=""/>
+<part name="L1" library="NSE LABS" deviceset="L_0603" device="" value="47nH"/>
 <part name="C1" library="NSE LABS" deviceset="C_0603" device="" value="47nF"/>
 <part name="C2" library="NSE LABS" deviceset="C_0603" device="" value="47pF"/>
 <part name="SUPPLY11" library="supply2" library_urn="urn:adsk.eagle:library:372" deviceset="GND" device=""/>
 <part name="SUPPLY12" library="supply2" library_urn="urn:adsk.eagle:library:372" deviceset="GND" device=""/>
-<part name="Y1" library="NSE LABS" deviceset="XTAL_SMD2016-4P" device=""/>
+<part name="Y1" library="NSE LABS" deviceset="XTAL_SMD2016-4P" device="" value="32MHz"/>
 <part name="SUPPLY13" library="supply2" library_urn="urn:adsk.eagle:library:372" deviceset="GND" device=""/>
 <part name="C14" library="NSE LABS" deviceset="C_0402" device="" value="1uF"/>
