File: KiCad/CPU Development Board/CPU Development Board.kicad_sch (KiCad schematic)
At the start: 29 parts, among them J1 Micro USB, J2 Debug, J3 Power Select Jumper, J4 Conn_01x16_Pin, J5 Conn_01x16_Pin, J6 Boot Select, SW1 Reset, U1 STM32L151C8T6, U2 AMS1117-3.3, Y1 16 MHz

Commit message: Central subsystem design
Connections:
- no-connect marks 11 -> 10
Changed lines of the file:
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@@
   (no_connect (at 179.07 119.38))
   (no_connect (at 179.07 124.46))
-  (no_connect (at 189.23 101.6))
   (no_connect (at 179.07 121.92))
   (no_connect (at 191.77 119.38))
