File: KiCad/Combined Boards/Power Subsystem.kicad_sch (KiCad schematic)
At the start: 0 parts

Commit message: Added solar charging circuit
Parts:
- added 82uH: L1, symbol Device:L
- added C1: 100 nF, symbol Device:C_Small
- added C2: 220 nF, symbol Device:C_Small
- added C3, C5: 10 uF, symbol Device:C_Polarized_Small_US
- added C4, C6: 4.7 uF, symbol Device:C_Small
- added C7: 470 nF, symbol Device:C_Small
- added D1, D2: SS54, symbol Device:D_Schottky
- added J1: Solar Panel, symbol Connector:Conn_01x02_Pin
- added J2: Charge Status, symbol Connector:Conn_01x02_Pin
- added J3: MPPT Resistors, symbol Connector:Conn_01x03_Pin
- added J4: Battery, symbol Connector:Conn_01x02_Pin
- added Q1: SI2301CDS-T1-GE3, Package_TO_SOT_SMD:SOT-23, symbol Transistor_FET:Si2319CDS
- added R1: 120, symbol Device:R_Small_US
- added R2: 1.02 ohm, symbol Device:R_Small_US
- added U1: ~, symbol Wireless Sensors:CN3791
Connections:
- new net: 82uH.2, R2.1, U1.8 (CSP)
- new net: C3.1, C4.1, J4.1 (Pin_1), R2.2, U1.7 (BAT)
- new net: 82uH.1, D1.1 (K), D2.1 (K)
- new net: R1.1, U1.5 (COM)
- new net: C2.1, R1.2
- new net: J2.1 (Pin_1), U1.3 (CHRG)
- new net: J2.2 (Pin_2), U1.4 (DONE)
- new net: C1.2, U1.1 (VG)
- new net: Q1.1 (G), U1.10 (DRV)
- new net: J3.2 (Pin_2), U1.6 (MPPT)
- new net: D1.2 (A), Q1.3 (D)
- new net GND: C2.2, C3.2, C4.2, C5.2, C6.2, C7.2, D2.2 (A), J1.2 (Pin_2), J3.3 (Pin_3), J4.2 (Pin_2), U1.2 (GND)
- new net VDC: C1.1, C5.1, C6.1, C7.1, J1.1 (Pin_1), J3.1 (Pin_1), Q1.2 (S), U1.9 (VCC)
Other:
- note added: "+"
- note added: "-"
- note added: "CHRG"
- note added: "DONE"

Commit message: Further work on power subsystem
Parts:
- removed J3: MPPT Resistors, symbol Connector:Conn_01x03_Pin
- added C8, C9: 1 uF, symbol Device:C_Small
- added D3: SS54, symbol Device:D_Schottky
- added J5: 3.3V, symbol Connector:Conn_01x02_Pin
- added Q1: SI2301CDS-T1-GE3, Package_TO_SOT_SMD:SOT-23, symbol Transistor_FET:Si2319CDS
- added R3, R4: None, symbol Device:R_Small_US
- added R5: 10K, symbol Device:R_Small_US
- added U2: XC6210B332MR, Package_TO_SOT_SMD:SOT-23-5, symbol Regulator_Linear:XC6210B332MR
- R2: value 1.02 ohm -> 1.02
- renumbered 82uH to 100uH
Connections:
- net GND: now also C8.2, C9.2, J5.2 (Pin_2), R4.2, R5.2, U2.2 (GND)
- net VDC: now also D3.2 (A), Q1.1 (G), R3.1, R5.1
- net at C3.1, C4.1, J4.1 (Pin_1)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: now also Q1.3 (D)
- net at U1.6 (MPPT): now also R3.2, R4.1
- new net: C9.1, J5.1 (Pin_1), U2.5 (VOUT)
- new net: C8.1, D3.1 (K), Q1.2 (S), U2.1 (VIN), U2.3 (CE)
Other:
- note added: "Through-hole resistors Include in layout but do not populate"

Commit message: More work on power subsystem
Parts:
- removed C8, C9: 1 uF, symbol Device:C_Small
- removed U2: XC6210B332MR, Package_TO_SOT_SMD:SOT-23-5, symbol Regulator_Linear:XC6210B332MR
- added C10, C11: 100 nF, symbol Device:C_Small
- added C8, C9: 10 uF, symbol Device:C_Polarized_Small_US
- added U2: HT7333-1, Package_TO_SOT_SMD:SOT-89-3, symbol Regulator_Linear:HT75xx-1-SOT89
- J5: value 3.3V -> 3.3V Out
Connections:
- net GND: now also C10.2, C11.2, C8.2, C9.2, U2.1 (GND)
- net at J5.1 (Pin_1): now also C11.1, C9.1, U2.3 (VOUT)
- net at D3.1 (K), Q1.2 (S): now also C10.1, C8.1, U2.2 (VIN)
Other:
- moved on the sheet: J5
