File: KiCad/Combined Boards/Power Subsystem.kicad_sch (KiCad schematic)
At the start: 34 parts, among them J1 Solar Panel, J2 Charge Status, J3 3.3V Out, J4 Battery, J5 Micro USB, Q1 SI2301CDS-T1-GE3, U2 HT7333-1

Commit message: Development version of power subsystem
Parts:
- added D4, D5: SS54, symbol Device:D_Schottky
Connections:
- net GND: now also J5.5 (GND)
- net VDC: now also D4.1 (K), D5.1 (K); no longer J1.1 (Pin_1)
- net at J5.1 (VBUS): now also D4.2 (A)
- new net: D5.2 (A), J1.1 (Pin_1)
- no-connect marks 5 -> 7
Other:
- note added: "Through-hole resistors. Include in layout but do not populate. Resistor values are based on the MPP voltage of the solar panel."
- note removed: "Through-hole resistors. Include in layout but do not populate. Resistor values are based the MPP voltage of the solar panel."
- title: Power Subsystem -> Power Subsystem Development Board
- moved on the sheet: J1, J5
Changed lines of the file:
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@@
   (paper "USLetter")
   (title_block
-    (title "Power Subsystem")
-    (date "2023-07-13")
+    (title "Power Subsystem Development Board")
+    (date "2023-08-01")
     (rev "A.1")
     (company "NSE Labs")
@@
   (junction (at 223.52 74.93) (diameter 0) (color 0 0 0 0)
   )
-  (no_connect (at 45.72 52.07))
-  (no_connect (at 35.56 57.15))
+  (no_connect (at 40.64 57.15))
+  (no_connect (at 40.64 59.69))
+  (no_connect (at 40.64 62.23))
+  (no_connect (at 30.48 67.31))
   (no_connect (at 176.53 106.68))
   (no_connect (at 196.85 106.68))
@@
     (stroke (width 0) (type default))
   )
+  (wire (pts (xy 33.02 87.63) (xy 36.83 87.63))
+    (stroke (width 0) (type default))
+  )
   (wire (pts (xy 119.38 95.25) (xy 121.92 95.25))
     (stroke (width 0) (type default))
@@
     (stroke (width 0) (type default))
   )
-  (wire (pts (xy 39.37 87.63) (xy 52.07 87.63))
-    (stroke (width 0) (type default))
-  )
   (wire (pts (xy 207.01 109.22) (xy 207.01 123.19))
     (stroke (width 0) (type default))
@@
     (stroke (width 0) (type default))
   )
-  (wire (pts (xy 43.18 90.17) (xy 43.18 93.98))
+  (wire (pts (xy 34.29 90.17) (xy 34.29 93.98))
+    (stroke (width 0) (type default))
+  )
+  (wire (pts (xy 52.07 52.07) (xy 52.07 72.39))
     (stroke (width 0) (type default))
   )
@@
     (stroke (width 0) (type default))
   )
+  (wire (pts (xy 52.07 80.01) (xy 52.07 87.63))
+    (stroke (width 0) (type default))
+  )
   (wire (pts (xy 146.05 85.09) (xy 146.05 86.36))
     (stroke (width 0) (type default))
@@
     (stroke (width 0) (type default))
   )
+  (wire (pts (xy 33.02 67.31) (xy 33.02 60.96))
+    (stroke (width 0) (type default))
+  )
   (wire (pts (xy 200.66 106.68) (xy 207.01 106.68))
     (stroke (width 0) (type default))
   )
-  (wire (pts (xy 39.37 90.17) (xy 43.18 90.17))
+  (wire (pts (xy 33.02 90.17) (xy 34.29 90.17))
     (stroke (width 0) (type default))
   )
@@
     (stroke (width 0) (type default))
   )
+  (wire (pts (xy 40.64 52.07) (xy 52.07 52.07))
+    (stroke (width 0) (type default))
+  )
   (wire (pts (xy 149.86 74.93) (xy 146.05 74.93))
     (stroke (width 0) (type default))
@@
     (stroke (width 0) (type default))
   )
+  (wire (pts (xy 251.46 102.87) (xy 251.46 106.68))
+    (stroke (width 0) (type default))
+  )
   (wire (pts (xy 73.66 87.63) (xy 83.82 87.63))
     (stroke (width 0) (type default))
   )
-  (wire (pts (xy 251.46 102.87) (xy 251.46 106.68))
-    (stroke (width 0) (type default))
-  )
   (wire (pts (xy 222.25 104.14) (xy 223.52 104.14))
     (stroke (width 0) (type default))
@@
     (stroke (width 0) (type default))
   )
+  (wire (pts (xy 44.45 87.63) (xy 52.07 87.63))
+    (stroke (width 0) (type default))
+  )
   (wire (pts (xy 87.63 95.25) (xy 83.82 95.25))
     (stroke (width 0) (type default))
@@
     (fill (type none))
   )
-  (text "-" (at 31.75 91.44 0)
+  (text "-" (at 25.4 91.44 0)
     (effects (font (size 1.27 1.27)) (justify left bottom))
   )
@@
     (effects (font (size 1.27 1.27)) (justify left bottom))
   )
-  (text "-" (at 259.08 99.06 0)
+  (text "-" (at 259.08 100.33 0)
     (effects (font (size 1.27 1.27)) (justify right bottom))
   )
@@
     (effects (font (size 1.27 1.27)) (justify right bottom))
   )
-  (text "Through-hole resistors.\nInclude in layout but\ndo not populate.\n\nResistor values are\nbased the MPP voltage\nof the solar panel."
+  (text "Through-hole resistors.\nInclude in layout but\ndo not populate.\n\nResistor values are\nbased on the MPP\nvoltage of the solar\npanel."
     (at 105.41 173.99 0)
     (effects (font (size 1.27 1.27)) (justify left bottom))
@@
     (effects (font (size 1.27 1.27)) (justify right bottom))
   )
-  (text "+" (at 31.75 87.63 0)
+  (text "+" (at 25.4 87.63 0)
     (effects (font (size 1.27 1.27)) (justify left bottom))
   )
@@
     )
   )
-  (symbol (lib_id "Connector:Conn_01x02_Pin") (at 34.29 87.63 0) (unit 1)
+  (symbol (lib_id "Connector:Conn_01x02_Pin") (at 27.94 87.63 0) (unit 1)
     (in_bom yes) (on_board yes) (dnp no)
-    (property "Reference" "J1" (at 29.21 88.9 0)
-      (effects (font (size 1.27 1.27)))
-    )
-    (property "Value" "Solar Panel" (at 33.02 85.09 0)
-      (effects (font (size 1.27 1.27)))
-    )
-    (property "Footprint" "" (at 34.29 87.63 0)
-      (effects (font (size 1.27 1.27)) hide)
-    )
-    (property "Datasheet" "~" (at 34.29 87.63 0)
+    (property "Reference" "J1" (at 22.86 88.9 0)
+      (effects (font (size 1.27 1.27)))
+    )
+    (property "Value" "Solar Panel" (at 26.67 85.09 0)
+      (effects (font (size 1.27 1.27)))
+    )
+    (property "Footprint" "" (at 27.94 87.63 0)
+      (effects (font (size 1.27 1.27)) hide)
+    )
+    (property "Datasheet" "~" (at 27.94 87.63 0)
       (effects (font (size 1.27 1.27)) hide)
     )
@@
     )
   )
-  (symbol (lib_id "Connector:USB_B_Micro") (at 38.1 46.99 0) (unit 1)
-    (in_bom yes) (on_board yes) (dnp no) (fields_autoplaced)
-    (property "Reference" "J5" (at 31.75 47.625 0)
+  (symbol (lib_id "Connector:USB_B_Micro") (at 33.02 57.15 0) (unit 1)
+    (in_bom yes) (on_board yes) (dnp no) (fields_autoplaced)
+    (property "Reference" "J5" (at 26.67 57.785 0)
       (effects (font (size 1.27 1.27)) (justify right))
     )
-    (property "Value" "Micro USB" (at 31.75 45.085 0)
+    (property "Value" "Micro USB" (at 26.67 55.245 0)
       (effects (font (size 1.27 1.27)) (justify right))
     )
-    (property "Footprint" "" (at 41.91 48.26 0)
-      (effects (font (size 1.27 1.27)) hide)
-    )
-    (property "Datasheet" "~" (at 41.91 48.26 0)
+    (property "Footprint" "" (at 36.83 58.42 0)
+      (effects (font (size 1.27 1.27)) hide)
+    )
+    (property "Datasheet" "~" (at 36.83 58.42 0)
       (effects (font (size 1.27 1.27)) hide)
     )
@@
     )
   )
-  (symbol (lib_id "power:GND") (at 43.18 93.98 0) (unit 1)
-    (in_bom yes) (on_board yes) (dnp no) (fields_autoplaced)
-    (property "Reference" "#PWR041" (at 43.18 100.33 0)
-      (effects (font (size 1.27 1.27)) hide)
-    )
-    (property "Value" "GND" (at 43.18 99.06 0)
-      (effects (font (size 1.27 1.27)) hide)
-    )
-    (property "Footprint" "" (at 43.18 93.98 0)
-      (effects (font (size 1.27 1.27)) hide)
-    )
-    (property "Datasheet" "" (at 43.18 93.98 0)
+  (symbol (lib_id "power:GND") (at 34.29 93.98 0) (unit 1)
+    (in_bom yes) (on_board yes) (dnp no) (fields_autoplaced)
+    (property "Reference" "#PWR041" (at 34.29 100.33 0)
+      (effects (font (size 1.27 1.27)) hide)
+    )
+    (property "Value" "GND" (at 34.29 99.06 0)
+      (effects (font (size 1.27 1.27)) hide)
+    )
+    (property "Footprint" "" (at 34.29 93.98 0)
+      (effects (font (size 1.27 1.27)) hide)
+    )
+    (property "Datasheet" "" (at 34.29 93.98 0)
       (effects (font (size 1.27 1.27)) hide)
     )
@@
         (path "/819f9f2e-5083-42df-b63a-6cdcb84600f5/f7d938fe-a9e3-47ad-82ab-29dd717a03fc"
           (reference "#PWR041") (unit 1)
+        )
+      )
+    )
+  )
+  (symbol (lib_id "Device:D_Schottky") (at 52.07 76.2 90) (unit 1)
+    (in_bom yes) (on_board yes) (dnp no) (fields_autoplaced)
+    (property "Reference" "D4" (at 54.61 75.8825 90)
+      (effects (font (size 1.27 1.27)) (justify right))
+    )
+    (property "Value" "SS54" (at 54.61 78.4225 90)
+      (effects (font (size 1.27 1.27)) (justify right))
+    )
+    (property "Footprint" "" (at 52.07 76.2 0)
+      (effects (font (size 1.27 1.27)) hide)
+    )
+    (property "Datasheet" "~" (at 52.07 76.2 0)
+      (effects (font (size 1.27 1.27)) hide)
+    )
+    (pin "1")
+    (pin "2")
+    (instances
+      (project "Combined Boards"
+        (path "/819f9f2e-5083-42df-b63a-6cdcb84600f5/f7d938fe-a9e3-47ad-82ab-29dd717a03fc"
+          (reference "D4") (unit 1)
         )
       )
@@
     )
   )
+  (symbol (lib_id "power:GND") (at 33.02 60.96 0) (unit 1)
+    (in_bom yes) (on_board yes) (dnp no) (fields_autoplaced)
+    (property "Reference" "#PWR062" (at 33.02 67.31 0)
+      (effects (font (size 1.27 1.27)) hide)
+    )
+    (property "Value" "GND" (at 33.02 66.04 0)
+      (effects (font (size 1.27 1.27)) hide)
+    )
+    (property "Footprint" "" (at 33.02 60.96 0)
+      (effects (font (size 1.27 1.27)) hide)
+    )
+    (property "Datasheet" "" (at 33.02 60.96 0)
+      (effects (font (size 1.27 1.27)) hide)
+    )
+    (pin "1")
+    (instances
+      (project "Combined Boards"
+        (path "/819f9f2e-5083-42df-b63a-6cdcb84600f5/f7d938fe-a9e3-47ad-82ab-29dd717a03fc"
+          (reference "#PWR062") (unit 1)
+        )
+      )
+    )
+  )
   (symbol (lib_id "Device:C_Polarized_Small_US") (at 223.52 82.55 0) (unit 1)
     (in_bom yes) (on_board yes) (dnp no) (fields_autoplaced)
@@
         )
       )
+    )
+  )
+  (symbol (lib_id "Device:D_Schottky") (at 40.64 87.63 180) (unit 1)
+    (in_bom yes) (on_board yes) (dnp no) (fields_autoplaced)
+    (property "Reference" "D5" (at 40.9575 82.55 0)
+      (effects (font (size 1.27 1.27)))
+    )
+    (property "Value" "SS54" (at 40.9575 85.09 0)
+      (effects (font (size 1.27 1.27)))
+    )
+    (property "Footprint" "" (at 40.64 87.63 0)
+      (effects (font (size 1.27 1.27)) hide)
+    )
+    (property "Datasheet" "~" (at 40.64 87.63 0)
+      (effects (font (size 1.27 1.27)) hide)
+    )
+    (pin "1")
+    (pin "2")
+    (instances
+      (project "Combined Boards"
+        (path "/819f9f2e-5083-42df-b63a-6cdcb84600f5/f7d938fe-a9e3-47ad-82ab-29dd717a03fc"
+          (reference "D5") (unit 1)
+        )
+      )
