File: KiCad/Combined Boards/Power Subsystem.kicad_sch (KiCad schematic)
At the start: 34 parts, among them J5 Solar Panel, J6 Micro USB, J8 Battery, Q1 SI2301CDS-T1-GE3, U5 HT7333-1

Commit message: Refined combined board design
Parts:
- added D6: 1N4148, Diode_THT:D_DO-35_SOD27_P7.62mm_Horizontal, symbol Diode:1N4148
- L8: renamed from 100uH1; value L1 -> 100uH
- renumbered J5 to J7, J6 to J8, J8 to J9
Connections:
- net VDC: now also D6.2 (A); no longer Q1.1 (G), R7.1
- new net: D6.1 (K), Q1.1 (G), R7.1
