File: KiCad/Combined Boards/Central Subsystem.kicad_sch (KiCad schematic)
At the start: 42 parts, among them J1 Antenna, J2 GPIO, J3 Debug, J4 Signal debug, J7 STEMMA QT, J9 Power, Q1 SI2301CDS-T1-GE3, SW1 Power, U2 STM32WLE5CCU6, Y1 32 MHz

Commit message: Refined combined board design
Parts:
- removed C18: 4.7 uF, symbol Device:C_Small
- renumbered J7 to J2, J9 to J5, J2 to J6
