File: EAGLE/Power_Dev_revA/Power_Dev_revA.2.sch (EAGLE design)
At the start: 36 parts, among them J1 HEADER_2PIN, J2 HEADER_2PIN, J3 HEADER_2PIN, J4 HEADER_2PIN, J5 MICRO_USB_SMD, Q1 SI2301CDS-T1-GE3, Q2 SI2301CDS-T1-GE3, U1 CN3791, U2 DW01A-G, U4 FS8205A

Commit message: Power A.2
Added connector for battery
Parts:
- added J6: 53261-0271, NSE LABS:53261-0271
- U2: value DW01A-G -> (none); device NSE LABS:DW01A-G -> NSE LABS:LDO_SOT89
- U3: value (none) -> DW01A-G; device NSE LABS:LDO_SOT89 -> NSE LABS:DW01A-G
- renumbered J1 to SOLAR, J2 to STATUS, J3 to OUTPUT, J4 to BATTERY
Connections:
- net GND: now also U2.GND; no longer U3.GND
- net N$15: now also U3.CS; no longer U2.CS
- net N$16: now also U3.OC; no longer U2.OC
- net N$17: now also U3.OD; no longer U2.OD
- net N$18: now also J6.1, U3.GND; no longer U2.GND
- net N$19: now also U3.VCC; no longer U2.VCC
- net N$20: now also J6.2
- net N$6: now also U2.VO; no longer U3.VO
- net N$8: now also U2.VI; no longer U3.VI
