File: KiCad/Power Development Board/Power Subsystem development board.kicad_sch (KiCad schematic)
At the start: 34 parts, among them J5 Solar Panel, J6 Micro USB, J8 Battery, Q1 SI2301CDS-T1-GE3, U5 HT7333-1

Commit message: Updated combined board schematics
Parts:
- added J2: Charge Status, symbol Connector:Conn_01x02_Pin
- added J3: 3.3V Out, symbol Connector:Conn_01x02_Pin
- R3: renamed from R4; value 10K -> None
- R4: renamed from R5; value 10K -> None
- renumbered 100uH1 to 100uH, C26 to C1, C30 to C10, C34 to C11, C33 to C12, C25 to C2, C28 to C3, C29 to C4, C23 to C5, C24 to C6, C27 to C7, C31 to C8, C32 to C9, D3 to D1, D4 to D2, D5 to D3, D2 to D4, D1 to D5, J5 to J1, J8 to J4, J6 to J5, R3 to R1, R6 to R2, R7 to R5, R9 to R6, R8 to R7, U3 to U1, U5 to U2, U6 to U3
Connections:
- net GND: now also J3.2 (Pin_2)
- net +3.3V: no longer names the net of C11.1, C9.1, U2.3 (VOUT)
- net +3.3V: now also J3.1 (Pin_1)
- net CHRG: no longer names the net of U1.3 (CHRG)
- net CHRG: now also J2.1 (Pin_1)
- net DONE: no longer names the net of U1.4 (DONE)
- net DONE: now also J2.2 (Pin_2)
Other:
- note added: "CHRG"
- note added: "DONE"
- note added: "J1, J2, J3, and J4 are 0.1 inch spaced holes where pins can be soldered."
- note added: "Through-hole resistors. Include in layout but do not populate. Resistor values are based on the MPP voltage of the solar panel."
- note removed: "J5 and J8 are 0.1 inch spaced holes where pins can be soldered."
- note removed: "To Central Subsystem"
- title: Power Subsystem -> Power Subsystem Development Board
