File: EAGLE/CombinedBoard_revA/CombinedBoard_revA.1.sch (EAGLE design)
At the start: 80 parts, among them J1 U.FL-R-SMT-1_80_, J10 SM04B-SRSS-TB_LF__SN_, J11 HEADER_3PIN, J2 HEADER_5PIN, J2A HEADER_10PIN, J2B HEADER_10PIN, J3 DEBUG, J5 SOLAR, J6 S2B-PH-SM4-TB_LF__SN_, J7 SM04B-SRSS-TB_LF__SN_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

Commit message: Comstation revA.1 error fix
fixed Y1 footprint
Parts:
- Y1: device NSE LABS:XTAL_SMD3225-4P -> NSE LABS:XTAL_SMD2016-4P
Changed lines of the file:
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@@
 <part name="C17" library="NSE LABS" deviceset="C_0402" device="" value="100nF"/>
 <part name="SUPPLY2" library="supply2" library_urn="urn:adsk.eagle:library:372" deviceset="GND" device=""/>
-<part name="Y1" library="NSE LABS" deviceset="XTAL_SMD3225-4P" device="" value="32MHz"/>
+<part name="Y1" library="NSE LABS" deviceset="XTAL_SMD2016-4P" device="" value="32MHz"/>
 <part name="C10" library="NSE LABS" deviceset="C_0402" device="" value="10pF"/>
 <part name="C11" library="NSE LABS" deviceset="C_0402" device="" value="10pF"/>
